File: board/ALF-3AAA.sch (KiCad schematic (older format))
At the start: 17 parts, among them M1 CONN_2, M2 CONN_2, Q1 2N3904, Q2 2N3904, Q3 2N3906, Q4 2N3906, SW1 SWITCH_INV

Commit message: Change to 3 transistor configuration
Parts:
- removed D2: DIODE, symbol DIODE
- added Q5: 2N3904, symbol NPN
- added Q6: 2N3906, symbol PNP
- R3, R4: value 51k -> 100k
Connections:
- net GND: now reaches BT1.2 (-), D1.2 (K), M2.2 (PM), R2.2
- net GND: now also Q5.1 (E); no longer Q2.1 (E)
- net at M1.1 (P1), Q1.3 (C), Q2.3 (C): now also Q5.3 (C)
- net at M2.1 (P1), Q3.3 (C), Q4.3 (C): now also Q6.3 (C)
- net at M1.2 (PM), R1.1, R5.1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: now also Q6.1 (E); no longer Q3.1 (E)
- net at BT1.1 (+): now also SW1.2
- new net: Q2.1 (E), Q5.2 (B)
- new net: Q3.1 (E), Q6.2 (B)
Other:
- moved on the sheet: Q1, Q2, Q3
Changed lines of the file:
@@
-EESchema Schematic File Version 2  date Wed 12 Dec 2012 03:41:13 PM CST
+EESchema Schematic File Version 2  date Wed 20 Feb 2013 08:39:22 PM CST
 LIBS:power
 LIBS:device
@@
 LIBS:contrib
 LIBS:valves
+LIBS:ALF-3AAA-cache
 EELAYER 27 0
 EELAYER END
@@
 Sheet 1 1
 Title ""
-Date "11 dec 2012"
+Date "20 feb 2013"
 Rev ""
 Comp ""
@@
 L NPN Q2
 U 1 1 509CBC7D
-P 3250 2900
-F 0 "Q2" H 3250 2750 50  0000 R CNN
-F 1 "2N3904" H 3250 3050 50  0000 R CNN
-	1    3250 2900
+P 3050 2600
+F 0 "Q2" H 3050 2450 50  0000 R CNN
+F 1 "2N3904" H 3050 2750 50  0000 R CNN
+F 2 "" H 3050 2600 60  0001 C CNN
+F 3 "" H 3050 2600 60  0001 C CNN
+	1    3050 2600
 	1    0    0    -1
 $EndComp
@@
 L NPN Q1
 U 1 1 509CBC8C
-P 2750 2700
-F 0 "Q1" H 2750 2550 50  0000 R CNN
-F 1 "2N3904" H 2750 2850 50  0000 R CNN
-	1    2750 2700
+P 2750 2400
+F 0 "Q1" H 2750 2250 50  0000 R CNN
+F 1 "2N3904" H 2750 2550 50  0000 R CNN
+F 2 "" H 2750 2400 60  0001 C CNN
+F 3 "" H 2750 2400 60  0001 C CNN
+	1    2750 2400
 	1    0    0    -1
 $EndComp
@@
 F 0 "Q4" H 4500 2800 60  0000 R CNN
 F 1 "2N3906" H 4400 2850 60  0000 R CNN
+F 2 "" H 4500 2950 60  0001 C CNN
+F 3 "" H 4500 2950 60  0001 C CNN
 	1    4500 2950
 	-1   0    0    1
@@
 L PNP Q3
 U 1 1 509CBCAA
-P 4200 2650
-F 0 "Q3" H 4200 2500 60  0000 R CNN
-F 1 "2N3906" H 4050 2500 60  0000 R CNN
-	1    4200 2650
+P 4200 2750
+F 0 "Q3" H 4200 2600 60  0000 R CNN
+F 1 "2N3906" H 4050 2600 60  0000 R CNN
+F 2 "" H 4200 2750 60  0001 C CNN
+F 3 "" H 4200 2750 60  0001 C CNN
+	1    4200 2750
 	-1   0    0    1
 $EndComp
 Wire Wire Line
-	2850 2900 3050 2900
-Wire Wire Line
-	2850 2500 2850 2400
-Wire Wire Line
-	2850 2400 3350 2400
-Wire Wire Line
-	3350 2150 3350 2700
-Connection ~ 3350 2400
-Wire Wire Line
-	4400 2650 4400 2750
-Wire Wire Line
-	4100 3500 4100 2850
-Wire Wire Line
-	4100 3250 4400 3250
-Wire Wire Line
-	4400 3250 4400 3150
-Connection ~ 4100 3250
-Wire Wire Line
 	3350 3100 3350 3950
 Wire Wire Line
 	3350 3500 3650 3500
 Wire Wire Line
-	3850 3500 4100 3500
+	3850 3500 4400 3500
 $Comp
 L CONN_2 M2
@@
 F 0 "M2" V 3700 3850 40  0000 C CNN
 F 1 "CONN_2" V 3800 3850 40  0000 C CNN
+F 2 "" H 3750 3850 60  0001 C CNN
+F 3 "" H 3750 3850 60  0001 C CNN
 	1    3750 3850
 	0    1    1    0
 $EndComp
-Wire Wire Line
-	4100 1550 4100 2450
 $Comp
 L CONN_2 M1
@@
 F 0 "M1" V 3700 1800 40  0000 C CNN
 F 1 "CONN_2" V 3800 1800 40  0000 C CNN
+F 2 "" H 3750 1800 60  0001 C CNN
+F 3 "" H 3750 1800 60  0001 C CNN
 	1    3750 1800
 	0    -1   -1   0
 $EndComp
 Wire Wire Line
-	3350 2150 3650 2150
+	3150 2150 3650 2150
 Wire Wire Line
 	4100 2150 3850 2150
@@
 P 4700 3350
 F 0 "R4" V 4780 3350 50  0000 C CNN
-F 1 "51k" V 4700 3350 50  0000 C CNN
+F 1 "100k" V 4700 3350 50  0000 C CNN
+F 2 "" H 4700 3350 60  0001 C CNN
+F 3 "" H 4700 3350 60  0001 C CNN
 	1    4700 3350
 	-1   0    0    1
@@
 P 2550 3100
 F 0 "R3" V 2630 3100 50  0000 C CNN
-F 1 "51k" V 2550 3100 50  0000 C CNN
+F 1 "100k" V 2550 3100 50  0000 C CNN
+F 2 "" H 2550 3100 60  0001 C CNN
+F 3 "" H 2550 3100 60  0001 C CNN
 	1    2550 3100
 	1    0    0    -1
@@
 F 0 "BT1" H 1600 3500 50  0000 C CNN
 F 1 "BATTERY" H 1600 3110 50  0000 C CNN
+F 2 "" H 1600 3300 60  0001 C CNN
+F 3 "" H 1600 3300 60  0001 C CNN
 	1    1600 3300
 	0    1    1    0
 $EndComp
-Wire Wire Line
-	2550 2850 2550 2700
 Wire Wire Line
 	1600 3950 5050 3950
@@
 F 0 "R1" V 2130 2400 50  0000 C CNN
 F 1 "LDR 1M" V 2050 2400 50  0000 C CNN
+F 2 "" H 2050 2400 60  0001 C CNN
+F 3 "" H 2050 2400 60  0001 C CNN
 	1    2050 2400
 	1    0    0    -1
@@
 F 0 "R2" V 2130 3100 50  0000 C CNN
 F 1 "LDR 1M" V 2050 3100 50  0000 C CNN
+F 2 "" H 2050 3100 60  0001 C CNN
+F 3 "" H 2050 3100 60  0001 C CNN
 	1    2050 3100
 	1    0    0    -1
@@
 F 0 "R5" V 5130 2350 50  0000 C CNN
 F 1 "220" V 5050 2350 50  0000 C CNN
+F 2 "" H 5050 2350 60  0001 C CNN
+F 3 "" H 5050 2350 60  0001 C CNN
 	1    5050 2350
 	1    0    0    -1
@@
 F 0 "D1" H 5050 3200 50  0000 C CNN
 F 1 "LED" H 5050 3000 50  0000 C CNN
+F 2 "" H 5050 3100 60  0001 C CNN
+F 3 "" H 5050 3100 60  0001 C CNN
 	1    5050 3100
 	0    1    1    0
@@
 F 0 "SW1" H 1400 2400 50  0000 C CNN
 F 1 "SWITCH_INV" H 1450 2100 50  0000 C CNN
+F 2 "" H 1600 2250 60  0001 C CNN
+F 3 "" H 1600 2250 60  0001 C CNN
 	1    1600 2250
 	0    -1   -1   0
@@
 Wire Wire Line
 	1600 1650 1600 1550
-$Comp
-L DIODE D2
-U 1 1 50C76B3F
-P 1200 2900
-F 0 "D2" H 1200 3000 40  0000 C CNN
-F 1 "DIODE" H 1200 2800 40  0000 C CNN
-	1    1200 2900
-	0    -1   -1   0
-$EndComp
-Wire Wire Line
-	1600 3000 1350 3000
-Wire Wire Line
-	1350 3000 1350 3100
-Wire Wire Line
-	1350 3100 1200 3100
-Wire Wire Line
-	1600 2750 1350 2750
-Wire Wire Line
-	1350 2750 1350 2700
-Wire Wire Line
-	1350 2700 1200 2700
 $Comp
 L R R6
@@
 F 0 "R6" V 730 3350 50  0000 C CNN
 F 1 "R" V 650 3350 50  0000 C CNN
+F 2 "" H 650 3350 60  0001 C CNN
+F 3 "" H 650 3350 60  0001 C CNN
 	1    650  3350
 	1    0    0    -1
@@
 F 0 "R7" V 880 3350 50  0000 C CNN
 F 1 "R" V 800 3350 50  0000 C CNN
+F 2 "" H 800 3350 60  0001 C CNN
+F 3 "" H 800 3350 60  0001 C CNN
 	1    800  3350
 	1    0    0    -1
 $EndComp
+$Comp
+L NPN Q5
+U 1 1 5124B1F4
+P 3350 2800
+F 0 "Q5" H 3350 2650 50  0000 R CNN
+F 1 "2N3904" H 3350 2950 50  0000 R CNN
+F 2 "" H 3350 2800 60  0001 C CNN
+F 3 "" H 3350 2800 60  0001 C CNN
+	1    3350 2800
+	1    0    0    -1
+$EndComp
+$Comp
+L PNP Q6
+U 1 1 5124B1FA
+P 3900 2550
+F 0 "Q6" H 3900 2400 60  0000 R CNN
+F 1 "2N3906" H 3750 2400 60  0000 R CNN
+F 2 "" H 3900 2550 60  0001 C CNN
+F 3 "" H 3900 2550 60  0001 C CNN
+	1    3900 2550
+	-1   0    0    1
+$EndComp
+Wire Wire Line
+	2550 2850 2550 2400
+Wire Wire Line
+	3450 3000 3450 3100
+Wire Wire Line
+	3450 3100 3350 3100
+Wire Wire Line
+	3450 2600 3450 2400
+Wire Wire Line
+	3450 2400 3150 2400
+Wire Wire Line
+	3150 2400 3150 2150
+Wire Wire Line
+	3150 2200 2850 2200
+Connection ~ 3150 2200
+Wire Wire Line
+	4100 1550 4100 2350
+Wire Wire Line
+	4400 3500 4400 3150
+Wire Wire Line
+	4400 3150 4100 3150
+Wire Wire Line
+	4100 3150 4100 2950
+Wire Wire Line
+	4100 2950 3800 2950
+Wire Wire Line
+	3800 2950 3800 2750
+Wire Wire Line
+	4100 2350 3800 2350
+Wire Wire Line
+	1600 3000 1600 2750
+$Comp
+L GND #PWR01
+U 1 1 5124B92B
+P 2600 4150
+F 0 "#PWR01" H 2600 4150 30  0001 C CNN
+F 1 "GND" H 2600 4080 30  0001 C CNN
+F 2 "" H 2600 4150 60  0000 C CNN
+F 3 "" H 2600 4150 60  0000 C CNN
+	1    2600 4150
+	1    0    0    -1
+$EndComp
+Wire Wire Line
+	2600 4150 2600 3950
+Connection ~ 2600 3950
 $EndSCHEMATC
